Commit message: rtabmap error: occupancy grid

File: catkin_ws/src/my_robot/urdf/my_robot.xacro (robot description, xacro)
@@ -36,4 +36,10 @@
     <dynamics damping="1.0" friction="1.0"/>
   </joint>
+  <!-- Optical camera joint -->
+  <joint name="camera_optical_joint" type="fixed">
+    <origin xyz="0 0 0" rpy="-1.5707 0 -1.5707"/>
+    <child link="camera_optical"/>
+    <parent link="camera"/>
+  </joint>
   <!-- LiDAR joint -->
   <joint type="fixed" name="hokuyo_joint">
@@ -167,4 +173,6 @@
     </visual>
   </link>
+  <!-- Optical Camera -->
+  <link name="camera_optical"></link>
   <!-- LiDAR -->
   <link name = "hokuyo">
