Commit message: finished robot package

File: catkin_ws/src/robot/urdf/dummy.xacro (robot description, xacro)
@@ -1,11 +1,6 @@
 <?xml version='1.0'?>
-<robot name="my_robot" xmlns:xacro="http://www.ros.org/wiki/xacro">
-  <!--
-    Plugins
-  -->
-  <xacro:include filename="$(find my_robot)/urdf/my_robot.gazebo" />
-  <!--
-    Robot Base
-  -->
+<robot name="dummy" xmlns:xacro="http://www.ros.org/wiki/xacro">
+  <!-- File containing the plugins -->
+  <xacro:include filename="$(find robot)/urdf/dummy.gazebo" />
   <link name="robot_footprint"></link>
   <joint name="robot_footprint_joint" type="fixed">
@@ -14,7 +9,7 @@
     <child link="chassis" />
   </joint>
-    Chassis
-  -->
+  <!-- Chassis -->
   <link name='chassis'>
+    <pose>0 0 0.1 0 0 0</pose>
     <inertial>
       <mass value="15.0"/>
@@ -23,6 +18,13 @@
           ixx="0.1" ixy="0" ixz="0"
           iyy="0.1" iyz="0"
-          izz="0.1" />
-    </inertial>
+          izz="0.1"
+      />
+    </inertial>
+    <visual name='chassis_visual'>
+      <origin xyz="0 0 0" rpy=" 0 0 0"/>
+      <geometry>
+        <box size=".4 .2 .1"/>
+      </geometry>
+    </visual>
     <collision name='collision'>
       <origin xyz="0 0 0" rpy=" 0 0 0"/>
@@ -31,10 +33,4 @@
       </geometry>
     </collision>
-    <visual name='chassis_visual'>
-      <origin xyz="0 0 0" rpy=" 0 0 0"/>
-      <geometry>
-        <box size=".4 .2 .1"/>
-      </geometry>
-    </visual>
     <collision name='back_caster_collision'>
       <origin xyz="-0.15 0 -0.05" rpy=" 0 0 0"/>
@@ -62,14 +58,7 @@
     </visual>
   </link>
-  <gazebo reference="chassis">
-    <material>Gazebo/Orange</material>
-  </gazebo>
-  <!--
-    Wheels
+  <!-- Left wheel
   -->
-  <!--
-    Left wheel
-  -->
-  <joint name="left_wheel_hinge" type="continuous">
+  <joint type="continuous" name="left_wheel_hinge">
     <origin xyz="0 0.15 0" rpy="0 0 0"/>
     <child link="left_wheel"/>
@@ -79,5 +68,5 @@
     <dynamics damping="1.0" friction="1.0"/>
   </joint>
-   <link name='left_wheel'>
+  <link name='left_wheel'>
     <inertial>
       <mass value="5.0"/>
@@ -86,5 +75,6 @@
           ixx="0.1" ixy="0" ixz="0"
           iyy="0.1" iyz="0"
-          izz="0.1" />
+          izz="0.1"
+      />
     </inertial>
     <collision name='left_wheel_collision'>
@@ -101,11 +91,7 @@
     </visual>
   </link>
-  <gazebo reference="left_wheel">
-    <material>Gazebo/DarkGrey</material>
-  </gazebo>
-  <!--
-    Right wheel
-  -->
-  <joint name="right_wheel_hinge" type="continuous">
+  <!-- Right wheel
+   -->
+  <joint type="continuous" name="right_wheel_hinge">
     <origin xyz="0 -0.15 0" rpy="0 0 0"/>
     <child link="right_wheel"/>
@@ -122,5 +108,6 @@
           ixx="0.1" ixy="0" ixz="0"
           iyy="0.1" iyz="0"
-          izz="0.1" />
+          izz="0.1"
+      />
     </inertial>
     <collision name='right_wheel_collision'>
@@ -137,15 +124,8 @@
     </visual>
   </link>
-  <gazebo reference="right_wheel">
-    <material>Gazebo/DarkGrey</material>
-  </gazebo>
-  <!--
-    Sensors
+  <!-- Camera
   -->
-  <!--
-    Camera
-  -->
-  <joint name="camera_joint" type="fixed">
-    <origin xyz="0.2 0 0" rpy="0 0 0"/>
+  <joint type="fixed" name="camera_joint">
+    <origin xyz="0.19 0 0.07" rpy="0 0 0"/>
     <child link="camera"/>
     <parent link="chassis"/>
@@ -154,5 +134,5 @@
     <dynamics damping="1.0" friction="1.0"/>
   </joint>
-  <link name="camera">
+  <link name = "camera">
     <inertial>
       <mass value="0.1"/>
@@ -174,11 +154,8 @@
       <origin xyz="0 0 0" rpy="0 0 0"/>
       <geometry>
-        <box size = "0.05 0.05 0.05"/>
-      </geometry>
-    </visual>
-  </link>
-  <gazebo reference="camera">
-    <material>Gazebo/Grey</material>
-  </gazebo>
+       <mesh filename="package://database/objects/models/camera/kinect.dae"/>
+      </geometry>
+    </visual>
+  </link>
   <joint name="camera_optical_joint" type="fixed">
     <origin xyz="0 0 0" rpy="-1.5707 0 -1.5707"/>
@@ -186,10 +163,10 @@
     <parent link="camera"/>
   </joint>
-  <link name="camera_optical"></link>
-  <!--
-    LiDAR
+  <link name="camera_optical">
+  </link>
+  <!-- LiDAR
   -->
   <joint type="fixed" name="hokuyo_joint">
-    <origin xyz="0.15 0 0.1" rpy="0 0 0"/>
+    <origin xyz="0.23 0 0" rpy="0 0 0"/>
     <child link="hokuyo"/>
     <parent link="chassis"/>
@@ -217,5 +194,5 @@
       <origin xyz="0 0 0" rpy="0 0 0"/>
       <geometry>
-       <mesh filename="package://my_robot/meshes/hokuyo.dae"/>
+       <mesh filename="package://database/objects/models/lidar/hokuyo.dae"/>
      </geometry>
     </visual>

Commit message: mesh update

File: catkin_ws/src/robot/urdf/dummy.xacro (robot description, xacro)
@@ -3,5 +3,169 @@
   <!-- File containing the plugins -->
   <xacro:include filename="$(find robot)/urdf/dummy.gazebo" />
-  <link name="robot_footprint"></link>
+  <!--
+  ******************************************************************************
+  All robot links
+  ******************************************************************************
+  -->
+  <!-- Link 0: Robot footprint -->
+  <link name="robot_footprint">
+    <!-- Empty -->
+  </link>
+  <!-- Link 1: Robot chassis -->
+  <link name='chassis'>
+    <pose>0 0 0.1 0 0 0</pose>
+    <inertial>
+      <mass value="15.0"/>
+      <origin xyz="0 0 0" rpy=" 0 0 0"/>
+      <inertia
+          ixx="0.1" ixy="0" ixz="0"
+          iyy="0.1" iyz="0"
+          izz="0.1"
+      />
+    </inertial>
+    <visual name='chassis_visual'>
+      <origin xyz="0 0 0" rpy=" 0 0 0"/>
+      <geometry>
+        <box size=".4 .2 .1"/>
+      </geometry>
+    </visual>
+    <collision name='chassis_collision'>
+      <origin xyz="0 0 0" rpy=" 0 0 0"/>
+      <geometry>
+        <box size=".4 .2 .1"/>
+      </geometry>
+    </collision>
+    <visual name='back_caster_visual'>
+      <origin xyz="-0.15 0 -0.05" rpy=" 0 0 0"/>
+      <geometry>
+        <sphere radius="0.05"/>
+      </geometry>
+    </visual>
+    <collision name='back_caster_collision'>
+      <origin xyz="-0.15 0 -0.05" rpy=" 0 0 0"/>
+      <geometry>
+        <sphere radius="0.0499"/>
+      </geometry>
+    </collision>
+    <visual name='front_caster_visual'>
+      <origin xyz="0.15 0 -0.05" rpy=" 0 0 0"/>
+      <geometry>
+        <sphere radius="0.05"/>
+      </geometry>
+    </visual>
+    <collision name='front_caster_collision'>
+      <origin xyz="0.15 0 -0.05" rpy=" 0 0 0"/>
+      <geometry>
+        <sphere radius="0.0499"/>
+      </geometry>
+    </collision>
+  </link>
+  <!-- Link 2: Left wheel -->
+  <link name='left_wheel'>
+    <inertial>
+      <mass value="5.0"/>
+      <origin xyz="0 0 0" rpy="0 1.5707 1.5707"/>
+      <inertia
+          ixx="0.1" ixy="0" ixz="0"
+          iyy="0.1" iyz="0"
+          izz="0.1"
+      />
+    </inertial>
+    <visual name='left_wheel_visual'>
+      <origin xyz="0 0 0" rpy="0 1.5707 1.5707"/>
+      <geometry>
+        <cylinder length="0.05" radius="0.1"/>
+      </geometry>
+    </visual>
+    <collision name='left_wheel_collision'>
+      <origin xyz="0 0 0" rpy="0 1.5707 1.5707"/>
+      <geometry>
+        <cylinder length="0.05" radius="0.1"/>
+      </geometry>
+    </collision>
+  </link>
+  <!-- Link 3: Right wheel -->
+  <link name='right_wheel'>
+    <inertial>
+      <mass value="5.0"/>
+      <origin xyz="0 0 0" rpy="0 1.5707 1.5707"/>
+      <inertia
+          ixx="0.1" ixy="0" ixz="0"
+          iyy="0.1" iyz="0"
+          izz="0.1"
+      />
+    </inertial>
+    <visual name='right_wheel_visual'>
+      <origin xyz="0 0 0" rpy="0 1.5707 1.5707"/>
+      <geometry>
+        <cylinder length="0.05" radius="0.1"/>
+      </geometry>
+    </visual>
+    <collision name='right_wheel_collision'>
+      <origin xyz="0 0 0" rpy="0 1.5707 1.5707"/>
+      <geometry>
+        <cylinder length="0.05" radius="0.1"/>
+      </geometry>
+    </collision>
+  </link>
+  <!-- Link 4: Camera RGB -->
+  <link name = "camera">
+    <inertial>
+      <mass value="0.1"/>
+      <origin xyz="0 0 0" rpy="0 0 0"/>
+      <inertia
+          ixx="1e-6" ixy="0" ixz="0"
+          iyy="1e-6" iyz="0"
+          izz="1e-6"
+      />
+      <box_inertia m="0.1" x="0.05" y="0.05" z="0.05"/>
+    </inertial>
+    <visual name='camera_visual'>
+      <origin xyz="0 0 0" rpy="0 0 0"/>
+      <geometry>
+       <mesh filename="package://database/objects/models/camera/kinect.dae"/>
+      </geometry>
+    </visual>
+    <collision name='camera_collision'>
+      <origin xyz="0 0 0" rpy="0 0 0"/>
+      <geometry>
+        <box size = "0.05 0.05 0.05"/>
+      </geometry>
+    </collision>
+  </link>
+  <!-- Link 4: Camera RGBD -->
+  <link name="camera_optical">
+    <!-- Empty -->
+  </link>
+  <!-- Link 5: Laser scanner -->
+  <link name = "hokuyo">
+    <inertial>
+      <mass value = "1e-5"/>
+      <origin xyz="0 0 0" rpy="0 0 0"/>
+      <inertia
+          ixx="1e-6" ixy="0" ixz="0"
+          iyy="1e-6" iyz="0"
+          izz="1e-6"
+      />
+    </inertial>
+    <visual name='hokuyo_visual'>
+      <origin xyz="0 0 0" rpy="0 0 0"/>
+      <geometry>
+       <mesh filename="package://database/objects/models/lidar/hokuyo.dae"/>
+     </geometry>
+    </visual>
+    <collision name='hokuyo_collision'>
+      <origin xyz="0 0 0" rpy="0 0 0"/>
+      <geometry>
+        <box size="0.1 0.1 0.1"/>
+      </geometry>
+    </collision>
+  </link>
+  <!--
+  ******************************************************************************
+  All robot joints
+  ******************************************************************************
+  -->
+  <!-- Footprint to chassis -->
   <joint name="robot_footprint_joint" type="fixed">
     <origin xyz="0 0 0" rpy="0 0 0" />
@@ -9,192 +173,36 @@
     <child link="chassis" />
   </joint>
-  <!-- Chassis -->
-  <link name='chassis'>
-    <pose>0 0 0.1 0 0 0</pose>
-    <inertial>
-      <mass value="15.0"/>
-      <origin xyz="0 0 0" rpy=" 0 0 0"/>
-      <inertia
-          ixx="0.1" ixy="0" ixz="0"
-          iyy="0.1" iyz="0"
-          izz="0.1"
-      />
-    </inertial>
-    <visual name='chassis_visual'>
-      <origin xyz="0 0 0" rpy=" 0 0 0"/>
-      <geometry>
-        <box size=".4 .2 .1"/>
-      </geometry>
-    </visual>
-    <collision name='collision'>
-      <origin xyz="0 0 0" rpy=" 0 0 0"/>
-      <geometry>
-        <box size=".4 .2 .1"/>
-      </geometry>
-    </collision>
-    <collision name='back_caster_collision'>
-      <origin xyz="-0.15 0 -0.05" rpy=" 0 0 0"/>
-      <geometry>
-        <sphere radius="0.0499"/>
-      </geometry>
-    </collision>
-    <visual name='back_caster_visual'>
-      <origin xyz="-0.15 0 -0.05" rpy=" 0 0 0"/>
-      <geometry>
-        <sphere radius="0.05"/>
-      </geometry>
-    </visual>
-    <collision name='front_caster_collision'>
-      <origin xyz="0.15 0 -0.05" rpy=" 0 0 0"/>
-      <geometry>
-        <sphere radius="0.0499"/>
-      </geometry>
-    </collision>
-    <visual name='front_caster_visual'>
-      <origin xyz="0.15 0 -0.05" rpy=" 0 0 0"/>
-      <geometry>
-        <sphere radius="0.05"/>
-      </geometry>
-    </visual>
-  </link>
-  <!-- Left wheel
-  -->
+  <!-- Chassis to wheels-->
   <joint type="continuous" name="left_wheel_hinge">
     <origin xyz="0 0.15 0" rpy="0 0 0"/>
+    <parent link="chassis"/>
     <child link="left_wheel"/>
-    <parent link="chassis"/>
     <axis xyz="0 1 0" rpy="0 0 0"/>
     <limit effort="10000" velocity="1000"/>
     <dynamics damping="1.0" friction="1.0"/>
   </joint>
-  <link name='left_wheel'>
-    <inertial>
-      <mass value="5.0"/>
-      <origin xyz="0 0 0" rpy="0 1.5707 1.5707"/>
-      <inertia
-          ixx="0.1" ixy="0" ixz="0"
-          iyy="0.1" iyz="0"
-          izz="0.1"
-      />
-    </inertial>
-    <collision name='left_wheel_collision'>
-      <origin xyz="0 0 0" rpy="0 1.5707 1.5707"/>
-      <geometry>
-        <cylinder length="0.05" radius="0.1"/>
-      </geometry>
-    </collision>
-    <visual name='left_wheel_visual'>
-      <origin xyz="0 0 0" rpy="0 1.5707 1.5707"/>
-      <geometry>
-        <cylinder length="0.05" radius="0.1"/>
-      </geometry>
-    </visual>
-  </link>
-  <!-- Right wheel
-   -->
   <joint type="continuous" name="right_wheel_hinge">
     <origin xyz="0 -0.15 0" rpy="0 0 0"/>
+    <parent link="chassis"/>
     <child link="right_wheel"/>
-    <parent link="chassis"/>
     <axis xyz="0 1 0" rpy="0 0 0"/>
     <limit effort="10000" velocity="1000"/>
     <dynamics damping="1.0" friction="1.0"/>
   </joint>
-  <link name='right_wheel'>
-    <inertial>
-      <mass value="5.0"/>
-      <origin xyz="0 0 0" rpy="0 1.5707 1.5707"/>
-      <inertia
-          ixx="0.1" ixy="0" ixz="0"
-          iyy="0.1" iyz="0"
-          izz="0.1"
-      />
-    </inertial>
-    <collision name='right_wheel_collision'>
-      <origin xyz="0 0 0" rpy="0 1.5707 1.5707"/>
-      <geometry>
-        <cylinder length="0.05" radius="0.1"/>
-      </geometry>
-    </collision>
-    <visual name='right_wheel_visual'>
-      <origin xyz="0 0 0" rpy="0 1.5707 1.5707"/>
-      <geometry>
-        <cylinder length="0.05" radius="0.1"/>
-      </geometry>
-    </visual>
-  </link>
-  <!-- Camera
-  -->
+  <!-- Chassis to sensors -->
   <joint type="fixed" name="camera_joint">
     <origin xyz="0.19 0 0.07" rpy="0 0 0"/>
+    <parent link="chassis"/>
     <child link="camera"/>
-    <parent link="chassis"/>
-    <axis xyz="0 1 0" rpy="0 0 0"/>
-    <limit effort="10000" velocity="1000"/>
-    <dynamics damping="1.0" friction="1.0"/>
-  </joint>
-  <link name = "camera">
-    <inertial>
-      <mass value="0.1"/>
-      <origin xyz="0 0 0" rpy="0 0 0"/>
-      <inertia
-          ixx="1e-6" ixy="0" ixz="0"
-          iyy="1e-6" iyz="0"
-          izz="1e-6"
-      />
-      <box_inertia m="0.1" x="0.05" y="0.05" z="0.05"/>
-    </inertial>
-    <collision name='camera_collision'>
-      <origin xyz="0 0 0" rpy="0 0 0"/>
-      <geometry>
-        <box size = "0.05 0.05 0.05"/>
-      </geometry>
-    </collision>
-    <visual name='camera_visual'>
-      <origin xyz="0 0 0" rpy="0 0 0"/>
-      <geometry>
-       <mesh filename="package://database/objects/models/camera/kinect.dae"/>
-      </geometry>
-    </visual>
-  </link>
+  </joint>
   <joint name="camera_optical_joint" type="fixed">
     <origin xyz="0 0 0" rpy="-1.5707 0 -1.5707"/>
+    <parent link="camera"/>
     <child link="camera_optical"/>
-    <parent link="camera"/>
-  </joint>
-  <link name="camera_optical">
-  </link>
-  <!-- LiDAR
-  -->
+  </joint>
   <joint type="fixed" name="hokuyo_joint">
     <origin xyz="0.23 0 0" rpy="0 0 0"/>
+    <parent link="chassis"/>
     <child link="hokuyo"/>
-    <parent link="chassis"/>
-    <axis xyz="0 1 0" rpy="0 0 0"/>
-    <limit effort="10000" velocity="1000"/>
-    <dynamics damping="1.0" friction="1.0"/>
-  </joint>
-  <link name = "hokuyo">
-    <inertial>
-      <mass value = "1e-5"/>
-      <origin xyz="0 0 0" rpy="0 0 0"/>
-      <inertia
-          ixx="1e-6" ixy="0" ixz="0"
-          iyy="1e-6" iyz="0"
-          izz="1e-6"
-      />
-    </inertial>
-    <collision name='hokuyo_collision'>
-      <origin xyz="0 0 0" rpy="0 0 0"/>
-      <geometry>
-        <box size="0.1 0.1 0.1"/>
-      </geometry>
-    </collision>
-    <visual name='hokuyo_visual'>
-      <origin xyz="0 0 0" rpy="0 0 0"/>
-      <geometry>
-       <mesh filename="package://database/objects/models/lidar/hokuyo.dae"/>
-     </geometry>
-    </visual>
-  </link>
+  </joint>
 </robot>

Commit message: F001: updated robot chassis and wheels to mesh

File: catkin_ws/src/robot/urdf/dummy.xacro (robot description, xacro)
@@ -14,5 +14,5 @@
   <!-- Link 1: Robot chassis -->
   <link name='chassis'>
-    <pose>0 0 0.1 0 0 0</pose>
+    <pose>0 0 0.5 0 0 0</pose>
     <inertial>
       <mass value="15.0"/>
@@ -27,5 +27,8 @@
       <origin xyz="0 0 0" rpy=" 0 0 0"/>
       <geometry>
-        <box size=".4 .2 .1"/>
+        <mesh
+          scale="0.9 0.6 0.6"
+          filename="package://database/objects/models/robot/chassis.dae"
+        />
       </geometry>
     </visual>
@@ -73,7 +76,10 @@
     </inertial>
     <visual name='left_wheel_visual'>
-      <origin xyz="0 0 0" rpy="0 1.5707 1.5707"/>
-      <geometry>
-        <cylinder length="0.05" radius="0.1"/>
+      <origin xyz="0 0 0" rpy="0 0 0"/>
+      <geometry>
+        <mesh
+          scale="0.9 0.9 0.9"
+          filename="package://database/objects/models/robot/wheel.dae"
+        />
       </geometry>
     </visual>
@@ -97,7 +103,10 @@
     </inertial>
     <visual name='right_wheel_visual'>
-      <origin xyz="0 0 0" rpy="0 1.5707 1.5707"/>
-      <geometry>
-        <cylinder length="0.05" radius="0.1"/>
+      <origin xyz="0 0 0" rpy="0 0 0"/>
+      <geometry>
+        <mesh
+          scale="0.9 0.9 0.9"
+          filename="package://database/objects/models/robot/wheel.dae"
+        />
       </geometry>
     </visual>
@@ -140,4 +149,5 @@
   <!-- Link 5: Laser scanner -->
   <link name = "hokuyo">
+    <origin xyz="0 0 10" rpy="0 0 0"/>
     <inertial>
       <mass value = "1e-5"/>

Commit message: F001: updated robot collision boxes

File: catkin_ws/src/robot/urdf/dummy.xacro (robot description, xacro)
@@ -19,7 +19,7 @@
       <origin xyz="0 0 0" rpy=" 0 0 0"/>
       <inertia
-          ixx="0.1" ixy="0" ixz="0"
-          iyy="0.1" iyz="0"
-          izz="0.1"
+        ixx="0.1" ixy="0" ixz="0"
+        iyy="0.1" iyz="0"
+        izz="0.1"
       />
     </inertial>
@@ -36,9 +36,9 @@
       <origin xyz="0 0 0" rpy=" 0 0 0"/>
       <geometry>
-        <box size=".4 .2 .1"/>
+        <box size="0.4 0.2 0.15"/>
       </geometry>
     </collision>
     <visual name='back_caster_visual'>
-      <origin xyz="-0.15 0 -0.05" rpy=" 0 0 0"/>
+      <origin xyz="-0.12 0 -0.05" rpy=" 0 0 0"/>
       <geometry>
         <sphere radius="0.05"/>
@@ -46,5 +46,5 @@
     </visual>
     <collision name='back_caster_collision'>
-      <origin xyz="-0.15 0 -0.05" rpy=" 0 0 0"/>
+      <origin xyz="-0.12 0 -0.05" rpy=" 0 0 0"/>
       <geometry>
         <sphere radius="0.0499"/>
@@ -52,5 +52,5 @@
     </collision>
     <visual name='front_caster_visual'>
-      <origin xyz="0.15 0 -0.05" rpy=" 0 0 0"/>
+      <origin xyz="0.14 0 -0.05" rpy=" 0 0 0"/>
       <geometry>
         <sphere radius="0.05"/>
@@ -58,5 +58,5 @@
     </visual>
     <collision name='front_caster_collision'>
-      <origin xyz="0.15 0 -0.05" rpy=" 0 0 0"/>
+      <origin xyz="0.14 0 -0.05" rpy=" 0 0 0"/>
       <geometry>
         <sphere radius="0.0499"/>
@@ -70,7 +70,7 @@
       <origin xyz="0 0 0" rpy="0 1.5707 1.5707"/>
       <inertia
-          ixx="0.1" ixy="0" ixz="0"
-          iyy="0.1" iyz="0"
-          izz="0.1"
+        ixx="0.1" ixy="0" ixz="0"
+        iyy="0.1" iyz="0"
+        izz="0.1"
       />
     </inertial>
@@ -87,5 +87,5 @@
       <origin xyz="0 0 0" rpy="0 1.5707 1.5707"/>
       <geometry>
-        <cylinder length="0.05" radius="0.1"/>
+        <cylinder length="0.07" radius="0.1"/>
       </geometry>
     </collision>
@@ -97,7 +97,7 @@
       <origin xyz="0 0 0" rpy="0 1.5707 1.5707"/>
       <inertia
-          ixx="0.1" ixy="0" ixz="0"
-          iyy="0.1" iyz="0"
-          izz="0.1"
+        ixx="0.1" ixy="0" ixz="0"
+        iyy="0.1" iyz="0"
+        izz="0.1"
       />
     </inertial>
@@ -114,5 +114,5 @@
       <origin xyz="0 0 0" rpy="0 1.5707 1.5707"/>
       <geometry>
-        <cylinder length="0.05" radius="0.1"/>
+        <cylinder length="0.07" radius="0.1"/>
       </geometry>
     </collision>
@@ -122,4 +122,34 @@
     <inertial>
       <mass value="0.1"/>
+      <origin xyz="0 0 0" rpy="0 0 0"/>
+      <inertia
+        ixx="1e-6" ixy="0" ixz="0"
+        iyy="1e-6" iyz="0"
+        izz="1e-6"
+      />
+      <box_inertia m="0.1" x="0.05" y="0.05" z="0.05"/>
+    </inertial>
+    <visual name='camera_visual'>
+      <origin xyz="0 0 0" rpy="0 0 0"/>
+      <geometry>
+       <mesh filename="package://database/objects/models/camera/kinect.dae"/>
+      </geometry>
+    </visual>
+    <collision name='camera_collision'>
+      <origin xyz="0 0 0" rpy="0 0 0"/>
+      <geometry>
+        <box size = "0.06 0.28 0.05"/>
+      </geometry>
+    </collision>
+  </link>
+  <!-- Link 4: Camera RGBD -->
+  <link name="camera_optical">
+    <!-- Empty -->
+  </link>
+  <!-- Link 5: Laser scanner -->
+  <link name = "hokuyo">
+    <origin xyz="0 0 5" rpy="0 0 0"/>
+    <inertial>
+      <mass value = "1e-5"/>
       <origin xyz="0 0 0" rpy="0 0 0"/>
       <inertia
@@ -128,34 +158,4 @@
           izz="1e-6"
       />
-      <box_inertia m="0.1" x="0.05" y="0.05" z="0.05"/>
-    </inertial>
-    <visual name='camera_visual'>
-      <origin xyz="0 0 0" rpy="0 0 0"/>
-      <geometry>
-       <mesh filename="package://database/objects/models/camera/kinect.dae"/>
-      </geometry>
-    </visual>
-    <collision name='camera_collision'>
-      <origin xyz="0 0 0" rpy="0 0 0"/>
-      <geometry>
-        <box size = "0.05 0.05 0.05"/>
-      </geometry>
-    </collision>
-  </link>
-  <!-- Link 4: Camera RGBD -->
-  <link name="camera_optical">
-    <!-- Empty -->
-  </link>
-  <!-- Link 5: Laser scanner -->
-  <link name = "hokuyo">
-    <origin xyz="0 0 10" rpy="0 0 0"/>
-    <inertial>
-      <mass value = "1e-5"/>
-      <origin xyz="0 0 0" rpy="0 0 0"/>
-      <inertia
-          ixx="1e-6" ixy="0" ixz="0"
-          iyy="1e-6" iyz="0"
-          izz="1e-6"
-      />
     </inertial>
     <visual name='hokuyo_visual'>
@@ -168,5 +168,5 @@
       <origin xyz="0 0 0" rpy="0 0 0"/>
       <geometry>
-        <box size="0.1 0.1 0.1"/>
+        <box size="0.05 0.05 0.07"/>
       </geometry>
     </collision>
@@ -202,5 +202,5 @@
   <!-- Chassis to sensors -->
   <joint type="fixed" name="camera_joint">
-    <origin xyz="0.19 0 0.07" rpy="0 0 0"/>
+    <origin xyz="0.16 0 0.07" rpy="0 0 0"/>
     <parent link="chassis"/>
     <child link="camera"/>
@@ -212,5 +212,5 @@
   </joint>
   <joint type="fixed" name="hokuyo_joint">
-    <origin xyz="0.23 0 0" rpy="0 0 0"/>
+    <origin xyz="0.23 0 -0.05" rpy="0 0 0"/>
     <parent link="chassis"/>
     <child link="hokuyo"/>
